Commit message: Extend simple robot and add nav2 config and launch file

File: urdf/wheelchair.urdf (robot description, URDF)
Before this commit: robot wheelchair, 4 links, 3 joints
Links:
- removed link laser_link
- added link base_footprint
- added link base_scan; visual cylinder length=0.05 radius=0.05
- link base_link: mass None -> 5.0; geometry collision box size=0.4 0.3 0.2; visual box size=0.4 0.3 0.2
Joints:
- removed joint base_to_laser
- added joint base_footprint_joint: type fixed, parent base_link, child base_footprint, origin xyz=0 0 0 rpy=0 0 0
- added joint base_link_to_laser: type fixed, parent base_link, child base_scan, origin xyz=0.2 0 0.15 rpy=0 0 0
